File: kicad_source/OpenCyphalServoController12.kicad_pcb (KiCad board)
At the start: 2 copper layers, 81 x 57 mm, 94 parts, among them CN1 SM04B-SRSS-TB, CN10 GH_SM04B-GHS-TB, CN11 GH_SM04B-GHS-TB, CN12 Powerpole_2, CN13 DNI, CN14 DNI, CN2 CONN_02X03, CN3 CONN_02X03, CN4 CONN_02X03, CN5 CONN_02X03, CN6 CONN_02X03, CN7 CONN_02X03, CN8 SM04B-SRSS-TB, CN9 RASPBERRYPI_PICO, SW1 SPST, U1 24LC64, U2 MCP2515, U3 SN65HVD232, U4 RAA211650, Y1 16MHz

Commit message: updated some labels
Other:
- board text added: "SERVO00 SERVO01"
- board text added: "SERVO02 SERVO03"
- board text added: "SERVO04 SERVO05"
- board text added: "SERVO07 SERVO06"
- board text added: "SERVO09 SERVO08"
- board text added: "SERVO11 SERVO10"
- board text removed: "ANALOG0"
- board text removed: "ANALOG1"
- board text removed: "INPUT0"
- board text removed: "INPUT1"
- board text removed: "INPUT2"
- board text removed: "INPUT3"
- board text removed: "OUTPUT0"
- board text removed: "OUTPUT1"
- board text removed: "SERVO0"
- board text removed: "SERVO1"
- board text removed: "V_IN | GND"
Changed lines of the file:
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@@
   (title_block
     (title "OpenCyphalServoController12")
-    (date "2023-02-03")
+    (date "2023-03-27")
     (rev "0.1")
     (company "generationmake")
@@
     (effects (font (size 1 1) (thickness 0.25)) (justify mirror))
   )
-  (gr_text "V_IN | GND" (at 33 98) (layer "B.SilkS")
-    (effects (font (size 0.6 0.6) (thickness 0.15)) (justify mirror))
+  (gr_text "+" (at 109 98.5) (layer "B.SilkS")
+    (effects (font (size 2 2) (thickness 0.5)) (justify left mirror))
   )
-  (gr_text "ANALOG0" (at 37 97 90) (layer "B.SilkS")
-    (effects (font (size 0.6 0.6) (thickness 0.15)) (justify right mirror))
-  )
-  (gr_text "INPUT0" (at 36 97 90) (layer "B.SilkS")
-    (effects (font (size 0.6 0.6) (thickness 0.15)) (justify right mirror))
-  )
-  (gr_text "OUTPUT1" (at 29 98 90) (layer "B.SilkS")
-    (effects (font (size 0.6 0.6) (thickness 0.15)) (justify right mirror))
+  (gr_text "SERVO07\nSERVO06" (at 112.5 102.5) (layer "B.SilkS")
+    (effects (font (size 0.6 0.6) (thickness 0.15)) (justify left mirror))
   )
-  (gr_text "SERVO1" (at 37.1 101.1) (layer "B.SilkS")
+  (gr_text "SERVO00\nSERVO01" (at 129.5 60.5) (layer "B.SilkS")
     (effects (font (size 0.6 0.6) (thickness 0.15)) (justify left mirror))
   )
-  (gr_text "ANALOG1" (at 38 97 90) (layer "B.SilkS")
-    (effects (font (size 0.6 0.6) (thickness 0.15)) (justify right mirror))
+  (gr_text "SERVO11\nSERVO10" (at 129.5 102.5) (layer "B.SilkS")
+    (effects (font (size 0.6 0.6) (thickness 0.15)) (justify left mirror))
   )
-  (gr_text "SERVO0" (at 37 100.1) (layer "B.SilkS")
+  (gr_text "find data and documentation at\nhttps://github.com/generationmake/OpenCyphalServoController12" (at 139.7 87) (layer "B.SilkS")
     (effects (font (size 0.6 0.6) (thickness 0.15)) (justify left mirror))
   )
-  (gr_text "INPUT2" (at 34 97 90) (layer "B.SilkS")
-    (effects (font (size 0.6 0.6) (thickness 0.15)) (justify right mirror))
+  (gr_text "+" (at 70.5 61.5) (layer "B.SilkS")
+    (effects (font (size 2 2) (thickness 0.5)) (justify left mirror))
   )
-  (gr_text "find data and documentation at\nhttps://github.com/generationmake/OpenCyphalServoController12" (at 139.7 87) (layer "B.SilkS")
+  (gr_text "SERVO02\nSERVO03" (at 120.5 60.5) (layer "B.SilkS")
     (effects (font (size 0.6 0.6) (thickness 0.15)) (justify left mirror))
   )
-  (gr_text "OUTPUT0" (at 31 97 90) (layer "B.SilkS")
-    (effects (font (size 0.6 0.6) (thickness 0.15)) (justify right mirror))
+  (gr_text "SERVO04\nSERVO05" (at 111.5 60.5) (layer "B.SilkS")
+    (effects (font (size 0.6 0.6) (thickness 0.15)) (justify left mirror))
   )
-  (gr_text "INPUT3" (at 33 97 90) (layer "B.SilkS")
-    (effects (font (size 0.6 0.6) (thickness 0.15)) (justify right mirror))
+  (gr_text "+" (at 77.5 72) (layer "B.SilkS")
+    (effects (font (size 2 2) (thickness 0.5)) (justify left mirror))
   )
-  (gr_text "INPUT1" (at 35 97 90) (layer "B.SilkS")
-    (effects (font (size 0.6 0.6) (thickness 0.15)) (justify right mirror))
+  (gr_text "SERVO09\nSERVO08" (at 120.5 102.5) (layer "B.SilkS")
+    (effects (font (size 0.6 0.6) (thickness 0.15)) (justify left mirror))
   )
   (gr_text "UCANPHY\n Micro" (at 69.5 103) (layer "F.SilkS")
