File: kicad_source/CyphalServoController12-CAN.kicad_sch (KiCad schematic)
At the start: 48 parts, among them CN1 SM04B-SRSS-TB, CN2 CONN_02X03, CN3 CONN_02X03, CN4 CONN_02X03, CN5 CONN_02X03, CN6 CONN_02X03, CN7 CONN_02X03, CN8 SM04B-SRSS-TB, CN9 RASPBERRYPI_PICO, SW1 SPST, U1 24LC64

Commit message: renamed comments and labels in kicad project
Other:
- title: OpenCyphalServoController12 -> CyphalServoController12/CAN
Changed lines of the file:
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@@
   (paper "A4")
   (title_block
-    (title "OpenCyphalServoController12")
-    (date "2023-02-04")
+    (title "CyphalServoController12/CAN")
+    (date "2023-09-24")
     (rev "0.1")
     (company "generationmake")
