File: kicad_source/mcp2515.kicad_sch (KiCad schematic)
At the start: 14 parts, among them CN10 GH_SM04B-GHS-TB, CN11 GH_SM04B-GHS-TB, U2 MCP2515, U3 SN65HVD232, Y1 16MHz

Commit message: renamed comments and labels in kicad project
Other:
- title: OpenCyphalServoController12 -> CyphalServoController12/CAN
Changed lines of the file:
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@@
   (paper "A4")
   (title_block
-    (title "OpenCyphalServoController12")
-    (date "2023-02-04")
+    (title "CyphalServoController12/CAN")
+    (date "2023-09-24")
     (rev "0.1")
     (company "generationmake")
