File: kicad_source/power.kicad_sch (KiCad schematic)
At the start: 32 parts, among them CN12 Powerpole_2, CN13 DNI, CN14 DNI, U4 RAA211650

Commit message: renamed comments and labels in kicad project
Other:
- title: OpenCyphalServoController12 -> CyphalServoController12/CAN
Changed lines of the file:
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@@
   (paper "A4")
   (title_block
-    (title "OpenCyphalServoController12")
-    (date "2023-02-04")
+    (title "CyphalServoController12/CAN")
+    (date "2023-09-24")
     (rev "0.1")
     (company "generationmake")
